File: Hardware/DIY_Mouse.kicad_pcb (KiCad board)
At the start: 2 copper layers, 60 x 105 mm, 20 parts, among them SW1 Rotary Encoder w/Switch, U1 Arduino Pro Micro 3.3v, U2 PMW3389DM-T3QU, U3 XC6206P332MR-G

Commit message: Changed Pinout for Rotary encoder to hardware interupt pin. Updated README and CHANGELOG files
Connections:
- U1 pad JP7_4: /Rot A -> unconnected-(U1-D6-PadJP7_4)
- U1 pad JP7_7: unconnected-(U1-D3-PadJP7_7) -> /Rot A
Routing:
- net /Rot A: track 128.0 -> 133.6 mm
Changed lines of the file:
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@@
 			(layers "*.Cu" "*.Mask")
 			(remove_unused_layers no)
-			(net "/Rot A")
+			(net "unconnected-(U1-D6-PadJP7_4)")
 			(pinfunction "D6_JP7_4")
-			(pintype "bidirectional")
+			(pintype "bidirectional+no_connect")
 			(solder_mask_margin 0.102)
 		)
@@
 			(layers "*.Cu" "*.Mask")
 			(remove_unused_layers no)
-			(net "unconnected-(U1-D3-PadJP7_7)")
+			(net "/Rot A")
 			(pinfunction "D3_JP7_7")
-			(pintype "bidirectional+no_connect")
+			(pintype "bidirectional")
 			(solder_mask_margin 0.102)
 		)
@@
 	)
 	(segment
+		(start 148.12 124.25)
+		(end 151.685686 120.684314)
+		(width 0.2)
+		(layer "F.Cu")
+		(net "/Rot A")
+	)
+	(segment
 		(start 146.7 42.85)
 		(end 165.365685 42.85)
@@
 	)
 	(segment
-		(start 151.685686 116.63)
-		(end 148.12 116.63)
-		(width 0.2)
-		(layer "F.Cu")
-		(net "/Rot A")
-	)
-	(segment
 		(start 144.4 45.15)
 		(end 146.7 42.85)
@@
 		(width 0.2)
 		(layer "F.Cu")
+		(net "/Rot A")
+	)
+	(segment
+		(start 151.685686 120.684314)
+		(end 151.685686 116.63)
+		(width 0.2)
+		(layer "F.Cu")

Commit message: PCB v2, Shell 3d model
Parts:
- added G***: LOGO, LOGO, F.Cu at (160.5, 138.2)
- moved C7 0.52 mm to (133.6, 104.9)
- moved R2 0.52 mm to (132.7, 96.9)
- moved C10 0.52 mm to (136.5, 100.8)
- moved C9 0.52 mm to (133.5, 100.8)
- moved C8 0.52 mm to (136.6, 104.9)
- turned S1 to -90 degrees
- turned S2 to -90 degrees
Routing:
- net Net-(U1-D9): track 50.0 -> 64.2 mm
- net Net-(U1-D4): track 87.8 -> 98.0 mm
- net +3.3V: track 107.3 -> 108.6 mm

Commit message: updated readme and pcb
Parts:
- moved G*** 39.6 mm to (121.0, 135.8)
- moved U1 0.59 mm to (140.7, 124.8), turned to 0 degrees
Routing:
- net /MOSI: track 28.3 -> 99.6 mm, vias 2 -> 1
- net /Rot A: track 133.6 -> 77.5 mm
- net /MOT: track 105.6 -> 49.6 mm
- net /Rot Switch: track 63.0 -> 116.5 mm
- net Net-(U1-D9): track 64.2 -> 114.0 mm
- net /NCS: track 20.9 -> 58.7 mm, vias 0 -> 2
- net /MISO: track 31.6 -> 60.3 mm, vias 0 -> 4
- net +3.3V: track 108.6 -> 81.0 mm
- net /SCLK: track 37.3 -> 64.2 mm, vias 4 -> 2
- net Net-(U1-D4): track 98.0 -> 80.3 mm
- net /Rot B: track 112.7 -> 109.5 mm
Other:
- board size 60 x 105 mm -> 52 x 99 mm
