File: Hardware/DIY_Mouse.kicad_sch (KiCad schematic)
At the start: 0 parts

Commit message: Added symbols and footprints for components and created PCB schematic
Parts:
- added C1: 4.7uF, symbol Device:C
- added C10, C2, C3, C6, C8: 0.1uF, symbol Device:C
- added C4, C5, C7, C9: 10uF, symbol Device:C
- added R1: Potentiometer, symbol Simulation_SPICE:Potentiometer
- added R2: 13Ω, symbol Device:R
- added R3: 10kΩ, symbol Device:R
- added S1, S2: Mouse Switch Hotswap, D2FC-F-7N_100M_:SW_D2FC-F-7N_100M_, symbol D2FC-F-7N_100M_:D2FC-F-7N_100M_
- added SW1: RotaryEncoder_Switch, symbol Device:RotaryEncoder_Switch
- added U1: Arduino Pro Micro 3.3v, DEV-12587:MODULE_DEV-12587, symbol DEV-12587:DEV-12587
- added U2: PMW3389DM-T3QU, symbol PMW3360DM-T2QU:PMW3360DM-T2QU
- added U3: XC6206P332MR-G, Package_TO_SOT_SMD:SOT-23, symbol Regulator_Linear:APE8865N-19-HF-3
Connections:
- new net: C1.2, C2.1, U2.3 (VDDPIX)
- new net: S2.1, U1.JP7_1 (D9)
- new net: R2.2, U2.15 (LED_P)
- new net: S1.1, U1.JP7_6 (D4)
- new net +1.9V: C10.1, C3.2, C4.1, C9.2, R2.1, U2.4 (VDD), U3.2 (VO)
- new net +3.3V: C5.1, C6.2, C7.2, C8.1, R1.1, R3.1, U1.JP6_4 (VCC), U2.5 (VDDIO), U3.3 (VI)
- new net GND: C1.1, C10.2, C2.2, C3.1, C4.2, C5.2, C6.1, C7.1, C8.2, C9.1, R1.3, S1.2, S2.2, SW1.C, SW1.S1, U1.JP6_2 (GND), U1.JP7_10 (GND), U1.JP7_9 (GND), U2.8 (GND), U3.1 (GND)
- new net MISO: R3.2, U1.JP6_10 (MISO), U2.12 (MISO)
- new net MOSI: U1.JP6_11 (MOSI), U2.11 (MOSI)
- new net MOT: U1.JP7_8 (D2), U2.9 (MOTION)
- new net NCS: U1.JP6_12 (D10), U2.13 (~{CS})
- new net Pot: R1.2, U1.JP6_8 (A0)
- new net Rot A: SW1.A, U1.JP7_4 (D6)
- new net Rot B: SW1.B, U1.JP7_3 (D7)
- new net Rot Switch: SW1.S2, U1.JP7_2 (D8)
- new net SCLK: U1.JP6_9 (SCK), U2.10 (SCLK)
- no-connect marks 0 -> 10
Other:
- note added: "Potentiometer"

Commit message: Created PCB design and created GBR and DRL files
Parts:
- removed C4: 10uF, symbol Device:C
- removed R1: Potentiometer, symbol Simulation_SPICE:Potentiometer
- C1, C10, C2, C3, C5, C6, C7, C8, C9: footprint (none) -> Capacitor_SMD:C_0805_2012Metric_Pad1.18x1.45mm_HandSolder
- R2, R3: footprint (none) -> Resistor_SMD:R_0805_2012Metric_Pad1.20x1.40mm_HandSolder
- S1, S2: footprint D2FC-F-7N_100M_:SW_D2FC-F-7N_100M_ -> Custom_Footprints:SW_D2FC-F-7N_100M_
- SW1: footprint (none) -> Rotary_Encoder:RotaryEncoder_Alps_EC11E-Switch_Vertical_H20mm
- U1: footprint DEV-12587:MODULE_DEV-12587 -> Custom_Footprints:MODULE_DEV-12587
- U2: footprint (none) -> Custom_Footprints:PMW3360
Connections:
- net Pot: no longer names the net of U1.JP6_8 (A0)
- no-connect marks 10 -> 11
Other:
- note removed: "Potentiometer"

Commit message: Changed Pinout for Rotary encoder to hardware interupt pin. Updated README and CHANGELOG files
Parts:
- S1, S2: value Mouse Switch Hotswap -> Mouse Switch
- SW1: value RotaryEncoder_Switch -> Rotary Encoder w/Switch
Connections:
- net Rot A: now also U1.JP7_7 (D3); no longer U1.JP7_4 (D6)
Changed lines of the file:
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@@
 	)
 	(no_connect
-		(at 62.23 57.15)
+		(at 62.23 64.77)
 	)
 	(no_connect
@@
 	)
 	(label "Rot A"
-		(at 62.23 64.77 180)
+		(at 62.23 57.15 180)
 		(effects
 			(font
@@
 		(fields_autoplaced yes)
 		(property "Reference" "S2"
-			(at 40.64 80.01 0)
+			(at 40.64 67.31 0)
 			(show_name no)
 			(do_not_autoplace no)
@@
 			)
 		)
-		(property "Value" "Mouse Switch Hotswap"
-			(at 40.64 77.47 0)
+		(property "Value" "Mouse Switch"
+			(at 40.64 69.85 0)
 			(show_name no)
 			(do_not_autoplace no)
@@
 			)
 		)
-		(property "Value" "RotaryEncoder_Switch"
+		(property "Value" "Rotary Encoder w/Switch"
 			(at 124.46 39.37 0)
 			(show_name no)
@@
 		(fields_autoplaced yes)
 		(property "Reference" "S1"
-			(at 43.18 67.31 0)
+			(at 43.18 54.61 0)
 			(show_name no)
 			(do_not_autoplace no)
@@
 			)
 		)
-		(property "Value" "Mouse Switch Hotswap"
-			(at 43.18 64.77 0)
+		(property "Value" "Mouse Switch"
+			(at 43.18 57.15 0)
 			(show_name no)
 			(do_not_autoplace no)

Commit message: Updated PCB manufacture files
Parts:
- C1: LCSC Part # (none) -> C354262
- C10, C2, C3, C6, C8: LCSC Part # (none) -> C519981
- C5, C7, C9: LCSC Part # (none) -> C326595
- R2: LCSC Part # (none) -> C2933313
- R3: LCSC Part # (none) -> C881248
- S1, S2, SW1, U1, U2: now not fitted; now left out of the parts list
- U3: LCSC Part # (none) -> C49195704
