File: Hardware/v2/DIY_Mouse.kicad_pcb (KiCad board)
At the start: 2 copper layers, 52 x 99 mm, 21 parts, among them SW1 Rotary Encoder w/Switch, U1 Arduino Pro Micro 3.3v, U2 PMW3389DM-T3QU, U3 XC6206P332MR-G

Commit message: Updated v2 PCB
Parts:
- U3: value XC6206P332MR-G -> XC6206-1.8V
Changed lines of the file:
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@@
 			)
 		)
-		(property "Value" "XC6206P332MR-G"
+		(property "Value" "XC6206-1.8V"
 			(at 0 2.4 90)
 			(layer "F.Fab")
@@
 			)
 		)
-		(property "Datasheet" "http://www.tme.eu/fr/Document/ced3461ed31ea70a3c416fb648e0cde7/APE8865-3.pdf"
+		(property "Datasheet" ""
 			(at 0 0 90)
 			(layer "F.Fab")
@@
 			)
 		)
-		(property "Description" "300mA Low Dropout Voltage Regulator, Fixed Output 1.9V, SOT-23"
+		(property "Description" "1.8V LDO"
 			(at 0 0 90)
 			(layer "F.Fab")
@@
 		)
 		(property "Value" "PMW3389DM-T3QU"
-			(at -1.6002 9.5 0)
+			(at 0 10.5 0)
 			(layer "Dwgs.User")
 			(effects
