File: Hardware/v2/DIY_Mouse.kicad_sch (KiCad schematic)
At the start: 17 parts, among them SW1 Rotary Encoder w/Switch, U1 Arduino Pro Micro 3.3v, U2 PMW3389DM-T3QU, U3 XC6206P332MR-G

Commit message: Updated v2 PCB
Parts:
- U3: value XC6206P332MR-G -> XC6206-1.8V
Changed lines of the file:
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@@
 			)
 		)
-		(property "Value" "XC6206P332MR-G"
+		(property "Value" "XC6206-1.8V"
 			(at 138.43 105.41 0)
 			(show_name no)
