File: Hardware/v2 (wired)/DIY_Mouse.kicad_pcb (KiCad board)
At the start: 2 copper layers, 52 x 99 mm, 21 parts, among them SW1 Rotary Encoder w/Switch, U1 Arduino Pro Micro 3.3v, U2 PMW3389DM-T3QU, U3 XC6206-1.8V

Commit message: updated PCBs
Parts:
- moved R2 2.38 mm to (130.8, 98.3)
- moved C7 1.70 mm to (134.6, 106.3)
- moved C8 1.70 mm to (137.6, 106.3)
- moved C2 1.70 mm to (149.9, 96.2)
- moved C1 1.70 mm to (152.3, 96.2)
- moved C5 1.64 mm to (152.6, 87.5)
- moved C6 1.64 mm to (150.2, 87.5)
- moved C3 1.62 mm to (150.2, 91.7)
- moved C10 1.30 mm to (136.2, 102.0)
- moved C9 1.30 mm to (133.2, 102.0)
Routing:
- net GND: track 19.9 -> 24.4 mm, vias 6 -> 13
- net /+1.9V: track 34.8 -> 38.3 mm
- net /MOSI: track 99.6 -> 96.9 mm
- net Net-(U2-LED_P): track 3.13 -> 5.62 mm
- net /NCS: track 58.7 -> 60.6 mm
- net /Rot A: track 77.5 -> 79.3 mm
- net Net-(U2-VDDPIX): track 5.35 -> 7.16 mm
- net /Rot B: track 109.5 -> 111.1 mm
- net /Rot Switch: track 116.5 -> 117.8 mm
- net +3.3V: track 81.0 -> 82.2 mm
- added copper zone on F.Cu, net GND
