File: Hardware/v3 (wireless)/Mouse v3.kicad_pcb (KiCad board)
At the start: 2 copper layers, 48 x 66 mm, 21 parts, among them SW1 Scroll + Middle, U1 PMW3389, U3 XC6206-1.8V, U4 XIAO_ESP32C3

Commit message: updated PCBs
Parts:
- moved C7 3.70 mm to (123.6, 87.7), turned to 180 degrees
- moved C4 3.61 mm to (123.6, 85.0), turned to 180 degrees
- moved R1 3.40 mm to (151.6, 82.8), turned to 90 degrees
- moved C1 3.33 mm to (128.4, 88.2)
- moved C2 3.09 mm to (129.5, 91.5)
- moved C6 3.09 mm to (126.9, 91.5)
- moved R3 2.95 mm to (128.3, 96.5)
- moved C9 2.63 mm to (127.9, 82.3)
- moved C3 2.63 mm to (130.5, 82.3)
- moved C5 2.06 mm to (123.2, 96.3)
- moved C8 2.06 mm to (123.2, 93.8)
- moved R2 1.76 mm to (152.2, 105.6)
Routing:
- net Net-(U1-LED_P): track 3.06 -> 7.17 mm
- net Net-(U1-~{RESET}): track 3.19 -> 6.38 mm
- net Net-(U1-VDDPIX): track 5.57 -> 8.25 mm
- net GND: track 34.3 -> 36.8 mm, vias 29 -> 35
- net +1V8: track 46.3 -> 48.6 mm
- net +3V3: track 54.3 -> 56.7 mm
- net /Rot B: track 43.2 -> 45.3 mm
- net /Middle Click: track 55.3 -> 56.9 mm
- net /SCLK: track 29.7 -> 31.0 mm
- net /MISO: track 27.0 -> 28.0 mm
